File: Schematic/EM84_OLED/EM84_OLED-backups/EM84_OLED-2023-12-11_110548/EM84_OLED.kicad_sch (KiCad schematic)
At the start: 21 parts, among them J1 FFC6, J2 Pin header, U1 ATMEGA328P-AU, U2 MCP6001T-I/OT, U3 Display_OLED_0.91_I2C, U4 NCP1117-5.0_SOT223, Y1 16MHz 16pF

Commit message: Updated PCB layout
Other:
- company: Retronics - Bjørner Sandom -> (none)
- title: EM84 TuningIndicator, OLED board -> (none)
- moved on the sheet: R2
Changed lines of the file:
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@@
 (kicad_sch (version 20230121) (generator eeschema)
   (paper "A4")
-  (title_block
-    (title "EM84 TuningIndicator, OLED board")
-    (date "2023-12-11")
-    (company "Retronics - Bjørner Sandom")
-  )
   (junction (at 103.505 102.87) (diameter 0) (color 0 0 0 0)
   )
@@
     (stroke (width 0) (type default))
   )
-  (wire (pts (xy 194.945 107.315) (xy 194.945 107.95))
+  (wire (pts (xy 179.705 106.68) (xy 179.705 107.315))
     (stroke (width 0) (type default))
   )
@@
     (stroke (width 0) (type default))
   )
+  (wire (pts (xy 179.705 113.665) (xy 194.945 113.665))
+    (stroke (width 0) (type default))
+  )
   (wire (pts (xy 215.265 111.125) (xy 217.17 111.125))
     (stroke (width 0) (type default))
@@
     (stroke (width 0) (type default))
   )
-  (wire (pts (xy 194.945 113.03) (xy 194.945 113.665))
+  (wire (pts (xy 179.705 112.395) (xy 179.705 113.665))
     (stroke (width 0) (type default))
   )
@@
     )
   )
-  (symbol (lib_id "power:+5V") (at 194.945 107.315 0) (unit 1)
-    (in_bom yes) (on_board yes) (dnp no)
-    (property "Reference" "#PWR09" (at 194.945 111.125 0)
-      (effects (font (size 1.27 1.27)) hide)
-    )
-    (property "Value" "+5V" (at 194.945 103.505 0)
-      (effects (font (size 1.27 1.27)))
-    )
-    (property "Footprint" "" (at 194.945 107.315 0)
-      (effects (font (size 1.27 1.27)) hide)
-    )
-    (property "Datasheet" "" (at 194.945 107.315 0)
+  (symbol (lib_id "power:+5V") (at 179.705 106.68 0) (unit 1)
+    (in_bom yes) (on_board yes) (dnp no)
+    (property "Reference" "#PWR09" (at 179.705 110.49 0)
+      (effects (font (size 1.27 1.27)) hide)
+    )
+    (property "Value" "+5V" (at 179.705 102.87 0)
+      (effects (font (size 1.27 1.27)))
+    )
+    (property "Footprint" "" (at 179.705 106.68 0)
+      (effects (font (size 1.27 1.27)) hide)
+    )
+    (property "Datasheet" "" (at 179.705 106.68 0)
       (effects (font (size 1.27 1.27)) hide)
     )
@@
     )
   )
-  (symbol (lib_id "Device:R_Small") (at 194.945 110.49 0) (unit 1)
-    (in_bom yes) (on_board yes) (dnp no)
-    (property "Reference" "R2" (at 193.675 109.855 0)
+  (symbol (lib_id "Device:R_Small") (at 179.705 109.855 0) (unit 1)
+    (in_bom yes) (on_board yes) (dnp no)
+    (property "Reference" "R2" (at 178.435 109.22 0)
       (effects (font (size 1.27 1.27)) (justify right))
     )
-    (property "Value" "10kΩ" (at 193.675 111.76 0)
+    (property "Value" "10kΩ" (at 178.435 111.125 0)
       (effects (font (size 1.27 1.27)) (justify right))
     )
-    (property "Footprint" "Retronics_Passives:R_0603_1608Metric_Pad0.98x0.95mm_HandSolder" (at 194.945 110.49 0)
-      (effects (font (size 1.27 1.27)) hide)
-    )
-    (property "Datasheet" "~" (at 194.945 110.49 0)
-      (effects (font (size 1.27 1.27)) hide)
-    )
+    (property "Footprint" "Retronics_Passives:R_0603_1608Metric_Pad0.98x0.95mm_HandSolder" (at 179.705 109.855 0)
+      (effects (font (size 1.27 1.27)) hide)
+    )
+    (property "Datasheet" "~" (at 179.705 109.855 0)
+      (effects (font (size 1.27 1.27)) hide)
+    )
