File: Schematic/EM84_Base/EM84_Base.kicad_pcb (KiCad board)
At the start: 2 copper layers, 17.3 x 17.3 mm, 7 parts, among them J1 Noval, J2 Pin header

Commit message: Updated PCB layout
Changed lines of the file:
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@@
     (fp_line (start 1 0.6) (end -1 0.6)
       (stroke (width 0.1) (type solid)) (layer "F.Fab"))
-    (pad "1" smd roundrect (at -1.025 0 90) (size 1.15 1.4) (layers "F.Cu" "F.Paste" "F.Mask") (roundrect_rratio 0.217391)
+    (pad "1" smd roundrect (at -1.025 0 90) (size 1.15 1.4) (layers "F.Cu" "F.Paste" "F.Mask") (roundrect_rratio 0.2173913043)
       (net 3 "F1") (pintype "passive"))
-    (pad "2" smd roundrect (at 1.025 0 90) (size 1.15 1.4) (layers "F.Cu" "F.Paste" "F.Mask") (roundrect_rratio 0.217391)
+    (pad "2" smd roundrect (at 1.025 0 90) (size 1.15 1.4) (layers "F.Cu" "F.Paste" "F.Mask") (roundrect_rratio 0.2173913043)
       (net 5 "Net-(D1-A)") (pintype "passive"))
     (model "${KICAD7_3DMODEL_DIR}/Fuse.3dshapes/Fuse_0805_2012Metric.step"
@@
     (fp_line (start 1 0.6) (end -1 0.6)
       (stroke (width 0.1) (type solid)) (layer "F.Fab"))
-    (pad "1" smd roundrect (at -1.025 0 90) (size 1.15 1.4) (layers "F.Cu" "F.Paste" "F.Mask") (roundrect_rratio 0.217391)
+    (pad "1" smd roundrect (at -1.025 0 90) (size 1.15 1.4) (layers "F.Cu" "F.Paste" "F.Mask") (roundrect_rratio 0.2173913043)
       (net 4 "F2") (pintype "passive"))
-    (pad "2" smd roundrect (at 1.025 0 90) (size 1.15 1.4) (layers "F.Cu" "F.Paste" "F.Mask") (roundrect_rratio 0.217391)
+    (pad "2" smd roundrect (at 1.025 0 90) (size 1.15 1.4) (layers "F.Cu" "F.Paste" "F.Mask") (roundrect_rratio 0.2173913043)
       (net 6 "Net-(D2-A)") (pintype "passive"))
     (model "${KICAD7_3DMODEL_DIR}/Fuse.3dshapes/Fuse_0805_2012Metric.step"

Commit message: File cleanup
Parts:
- removed F2: T1A, Retronics_Passives:Fuse_0805_2012Metric_Pad1.15x1.40mm_HandSolder
- added FB1: 330Ω@100MHz, Retronics_Passives:L_0805_2012Metric_Pad1.15x1.40mm_HandSolder, F.Cu at (139.5, 83.2)
- F1: footprint Retronics_Passives:Fuse_0805_2012Metric_Pad1.15x1.40mm_HandSolder -> Retronics_Passives:Fuse_1206_3216Metric
- moved D1 5.16 mm to (141.4, 88.0)
- moved D2 5.16 mm to (139.5, 88.0)
- moved F1 4.15 mm to (141.7, 82.8)
Connections:
- D1 pad 1: VCC -> Net-(D1-K)
- D1 pad 2: Net-(D1-A) -> H1
- D2 pad 1: VCC -> Net-(D1-K)
- D2 pad 2: Net-(D2-A) -> H2
- F1 pad 1: F1 -> Net-(D1-K)
- F1 pad 2: Net-(D1-A) -> Net-(F1-Pad2)
- J1 pad 4: F1 -> H1
- J1 pad 5: F2 -> H2
Routing:
- net F1: track 11.0 -> 0.00 mm
- net H1: track 0.00 -> 9.77 mm
- net Net-(D1-K): track 0.00 -> 4.71 mm
- net Net-(F1-Pad2): track 0.00 -> 3.74 mm
- net F2: track 3.67 -> 0.00 mm
- net H2: track 0.00 -> 2.91 mm
- net VCC: track 11.1 -> 8.65 mm
- net Net-(D2-A): track 1.72 -> 0.00 mm
- net Net-(D1-A): track 1.72 -> 0.00 mm
Other:
- board size 17.3 x 17.3 mm -> 17.4 x 17.4 mm
- board text added: "GND VCC AGC"
- board text added: "locked"
- board text removed: "EM84_Base R0155_2350_Pb Bjørner Sandom"
- board text removed: "GND VCC SIG"
