File: Schematic/EM84_Base/EM84_Base.kicad_sch (KiCad schematic)
At the start: 7 parts, among them J1 Noval, J2 Pin header

Commit message: File cleanup
Parts:
- removed F2: T1A, Retronics_Passives:Fuse_0805_2012Metric_Pad1.15x1.40mm_HandSolder, symbol Device:Fuse
- added FB1: 330Ω@100MHz, Retronics_Passives:L_0805_2012Metric_Pad1.15x1.40mm_HandSolder, symbol Device:FerriteBead
- C1: value 1000µF 16V -> 1000µF 10V
- F1: footprint Retronics_Passives:Fuse_0805_2012Metric_Pad1.15x1.40mm_HandSolder -> Retronics_Passives:Fuse_1206_3216Metric
Connections:
- net F2 is gone; now on net H2: J1.5 (Pin_5)
- net VCC: now also FB1.2; no longer D1.1 (K), D2.1 (K)
- net H2: now reaches D2.2 (A)
- net at F1.2: now also FB1.1; no longer D1.2 (A)
- net F1: no longer names the net of F1.1
- net F1: now also D1.1 (K), D2.1 (K); no longer J1.4 (Pin_4)
- net SIG renamed AGC
- new net H1: D1.2 (A), J1.4 (Pin_4)
Other:
- moved on the sheet: C1, D1, D2, F1
