File: Schematic/EM84_OLED/EM84_OLED.kicad_pcb (KiCad board)
At the start: 2 copper layers, 47.7 x 15 mm, 22 parts, among them J1 FFC6, J2 Pin header, U1 ATMEGA328P-AU, U2 MCP6001T-I/OT, U3 Display_OLED_0.91_I2C, U4 NCP1117-5.0_SOT223, Y1 16MHz 16pF

Commit message: File cleanup
Parts:
- removed the R2 at (62.4, 83.8)
- added J2: EMI Shield, Retronics_Hardware:EMI_Shield_MS192-10S, B.Cu at (70.5, 70.1)
- added U3: NCP1117-5.0_SOT223, Retronics_IC_Power:SOT-223-3_TabPin2, B.Cu at (42.6, 74.0)
- C5: renamed from C8; value 1µF -> 10µF
- J1: renamed from J2; footprint Retronics_Connectors:PinHeader_1x03_P2.54mm_Horizontal -> Retronics_Connectors:PinHeader_1x03_P2.54mm_Horizontal_Alt
- U4: value NCP1117-5.0_SOT223 -> MCP130T-460I/TT; footprint Retronics_IC_Power:SOT-223-3_TabPin2 -> Package_TO_SOT_SMD:SOT-23
- moved U4 10.7 mm to (54.2, 74.1), turned to 90 degrees
- moved J3 10.6 mm to (77.8, 77.5), turned to -90 degrees
- moved C9 8.77 mm to (68.7, 75.3), turned to -90 degrees
- moved C10 8.71 mm to (67.5, 71.4), turned to 0 degrees
- moved C6 8.67 mm to (54.2, 80.3), turned to 0 degrees
- moved C4 6.03 mm to (59.7, 83.6)
- moved Y1 5.20 mm to (54.2, 82.8), turned to 180 degrees
- moved C1 5.18 mm to (63.1, 83.6)
- moved C7 5.18 mm to (63.1, 71.4)
- moved U2 5.10 mm to (61.6, 77.5)
- moved C2 4.74 mm to (58.4, 71.4)
- moved C5 4.50 mm to (45.2, 81.3), turned to 180 degrees
- moved R2 1.25 mm to (41.9, 83.0)
- moved R3 1.25 mm to (38.4, 83.0)
- moved G*** 1.11 mm to (46.3, 73.4)
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- renumbered C7 to C10, C6 to C3, C3 to C4, C4 to C6, C5 to C7, C10 to C8, J1 to J3, R3 to R2, R4 to R3, U2 to U1, U1 to U2, U3 to U5
Connections:
- net Net-(J2-Pin_3) renamed /AGC
- net V_TUNE renamed AGC_INV
- C4 pad 1: Net-(U1-XTAL1) -> Net-(U2-XTAL1)
- C6 pad 1: Net-(U1-XTAL2) -> Net-(U2-XTAL2)
- C9 pad 2: Net-(U1-~{RESET}) -> Net-(U2-~{RESET})
- J1 pad 2: Net-(J2-Pin_2) -> Net-(J1-Pin_2)
- U2 pad 29: Net-(U1-~{RESET}) -> Net-(U2-~{RESET})
- U2 pad 7: Net-(U1-XTAL1) -> Net-(U2-XTAL1)
- U2 pad 8: Net-(U1-XTAL2) -> Net-(U2-XTAL2)
- U4 pad 1: GND -> Net-(U2-~{RESET})
- U4 pad 3: Net-(J2-Pin_2) -> GND
- Y1 pad 1: Net-(U1-XTAL2) -> Net-(U2-XTAL1)
- Y1 pad 3: Net-(U1-XTAL1) -> Net-(U2-XTAL2)
Routing:
- net Net-(U2-~{RESET}): track 0.00 -> 16.4 mm, vias 0 -> 2
- net +5V: track 63.4 -> 75.6 mm
- net Net-(U1-~{RESET}): track 11.4 -> 0.00 mm, vias 2 -> 0
- net Net-(J1-Pin_2): track 0.00 -> 9.43 mm
- net Net-(J2-Pin_2): track 9.36 -> 0.00 mm
- net Net-(U1-XTAL2): track 8.47 -> 0.00 mm
- net GND: track 18.8 -> 27.2 mm, vias 17 -> 23
- net Net-(U2-XTAL2): track 0.00 -> 7.55 mm
- net AGC_INV: track 14.5 -> 21.2 mm
- net Net-(J3-Pin_4): track 10.1 -> 16.5 mm
- net Net-(U1-XTAL1): track 5.95 -> 0.00 mm
- net Net-(U2-XTAL1): track 0.00 -> 5.75 mm
- net SDA: track 14.0 -> 9.60 mm, vias 1 -> 2
- net SCL: track 12.6 -> 10.1 mm, vias 1 -> 0
- net Net-(R1-Pad1): track 7.14 -> 6.29 mm
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Other:
- board size 47.7 x 15 mm -> 47.5 x 15 mm
- board text added: "locked"
- board text removed: "EM84_Display R0156_2350_Pb Bjørner Sandom"
